File: GaN-LTC7891/GaN-LTC7891/GaN-LTC7891.kicad_sch (KiCad schematic)
At the start: 35 parts, among them IC1 LTC7891RUFDM#PBF

Commit message: Schematics for Si and GaN for LTC7800 controller
Parts:
- removed B_GANFET, T_GANFET: EPC2001C, EPC_FETs:D0188, symbol EPC_FETs:EPC2001C
- added Q1, Q2: EPC2066, EPC_FETs:D0650, symbol EPC_FETs:EPC2066
Connections:
- net GND: now also Q2.10 (S5), Q2.13 (S6), Q2.14 (S7), Q2.17 (S8), Q2.18 (S9), Q2.2 (S1), Q2.21 (S10), Q2.22 (S11), Q2.25 (S12), Q2.26 (S13), Q2.29 (S14), Q2.30 (Sub), Q2.5 (S2), Q2.6 (S3), Q2.9 (S4)
- net SW: now also Q1.10 (S5), Q1.13 (S6), Q1.14 (S7), Q1.17 (S8), Q1.18 (S9), Q1.2 (S1), Q1.21 (S10), Q1.22 (S11), Q1.25 (S12), Q1.26 (S13), Q1.29 (S14), Q1.30 (Sub), Q1.5 (S2), Q1.6 (S3), Q1.9 (S4), Q2.11 (D5), Q2.12 (D6), Q2.15 (D7), Q2.16 (D8), Q2.19 (D9), Q2.20 (D10), Q2.23 (D11), Q2.24 (D12), Q2.27 (D13), Q2.28 (D14), Q2.3 (D1), Q2.4 (D2), Q2.7 (D3), Q2.8 (D4)
- net VIN: now also Q1.11 (D5), Q1.12 (D6), Q1.15 (D7), Q1.16 (D8), Q1.19 (D9), Q1.20 (D10), Q1.23 (D11), Q1.24 (D12), Q1.27 (D13), Q1.28 (D14), Q1.3 (D1), Q1.4 (D2), Q1.7 (D3), Q1.8 (D4)
- net at R6.1, R7.1, TFET_VGS.2: now also Q1.1 (G)
- net at BFET_VGS.2, R8.2, R9.2: now also Q2.1 (G)
Changed lines of the file:
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@@
 	(paper "A4")
 	(junction
-		(at 54.61 123.19)
-		(diameter 0)
-		(color 0 0 0 0)
-	)
-	(junction
 		(at 68.58 115.57)
 		(diameter 0)
@@
 	)
 	(junction
-		(at 85.09 123.19)
-		(diameter 0)
-		(color 0 0 0 0)
-	)
-	(junction
 		(at 119.38 104.14)
 		(diameter 0)
@@
 	)
 	(junction
+		(at 85.09 123.19)
+		(diameter 0)
+		(color 0 0 0 0)
+	)
+	(junction
 		(at 139.7 101.6)
 		(diameter 0)
@@
 	)
 	(junction
+		(at 54.61 123.19)
+		(diameter 0)
+		(color 0 0 0 0)
+	)
+	(junction
 		(at 228.6 111.76)
 		(diameter 0)
@@
 	)
 	(symbol
+		(lib_id "EPC_FETs:EPC2066")
+		(at 85.09 115.57 270)
+		(mirror x)
+		(unit 1)
+		(exclude_from_sim no)
+		(in_bom yes)
+		(on_board yes)
+		(dnp no)
+		(property "Reference" "Q1"
+			(at 85.09 105.41 90)
+			(effects
+				(font
+					(size 1.27 1.27)
+				)
+			)
+		)
+		(property "Value" "EPC2066"
+			(at 85.09 107.95 90)
+			(effects
+				(font
+					(size 1.27 1.27)
+				)
+			)
+		)
+		(property "Footprint" "EPC_FETs:D0650"
+			(at 81.4324 109.6772 0)
+			(effects
+				(font
+					(size 1.27 1.27)
+				)
+				(hide yes)
+			)
+		)
+		(property "Datasheet" ""
+			(at 85.09 115.57 0)
+			(effects
+				(font
+					(size 1.27 1.27)
+				)
+				(hide yes)
+			)
+		)
+		(property "Description" "40V 1.1mE 90A"
+			(at 85.09 110.49 90)
+			(effects
+				(font
+					(size 1.27 1.27)
+				)
+			)
+		)
+		(pin "11"
+		)
+		(pin "1"
+		)
+		(pin "3"
+		)
+		(pin "23"
+		)
+		(pin "7"
+		)
+		(pin "24"
+		)
+		(pin "20"
+		)
+		(pin "4"
+		)
+		(pin "27"
+		)
+		(pin "19"
+		)
+		(pin "15"
+		)
+		(pin "28"
+		)
+		(pin "12"
+		)
+		(pin "16"
+		)
+		(pin "8"
+		)
+		(pin "10"
+		)
+		(pin "13"
+		)
+		(pin "14"
+		)
+		(pin "17"
+		)
+		(pin "18"
+		)
+		(pin "2"
+		)
+		(pin "21"
+		)
+		(pin "22"
+		)
+		(pin "25"
+		)
+		(pin "26"
+		)
+		(pin "29"
+		)
+		(pin "30"
+		)
+		(pin "5"
+		)
+		(pin "6"
+		)
+		(pin "9"
+		)
+		(instances
+			(project "GaN-LTC7891"
+				(path "/7f2baae8-823e-4e28-b900-0a7e85154029"
+					(reference "Q1")
+					(unit 1)
+				)
+			)
+		)
+	)
+	(symbol
 		(lib_id "Device:C")
 		(at 77.47 64.77 90)
@@
 	)
 	(symbol
-		(lib_id "EPC_FETs:EPC2001C")
-		(at 85.09 115.57 270)
-		(mirror x)
-		(unit 1)
-		(exclude_from_sim no)
-		(in_bom yes)
-		(on_board yes)
-		(dnp no)
-		(property "Reference" "T_GANFET"
-			(at 84.836 107.696 90)
-			(effects
-				(font
-					(size 1.27 1.27)
-				)
-				(justify left)
-			)
-		)
-		(property "Value" "EPC2001C"
-			(at 83.566 111.76 90)
-			(effects
-				(font
-					(size 1.27 1.27)
-				)
-				(justify left)
-			)
-		)
-		(property "Footprint" "EPC_FETs:D0188"
-			(at 81.4832 109.22 0)
-			(effects
-				(font
-					(size 1.27 1.27)
-					(color 0 0 194 1)
-				)
-				(hide yes)
-			)
-		)
-		(property "Datasheet" ""
-			(at 85.09 115.57 0)
-			(effects
-				(font
-					(size 1.27 1.27)
-				)
-				(hide yes)
-			)
-		)
-		(property "Description" "100V 7mE 36A"
-			(at 83.566 109.728 90)
-			(effects
-				(font
-					(size 1.27 1.27)
-					(color 0 0 194 1)
-				)
-				(justify left)
-			)
-		)
-		(pin "6"
-		)
-		(pin "4"
-		)
-		(pin "2"
-		)
-		(pin "8"
-		)
-		(pin "3"
-		)
-		(pin "11"
-		)
-		(pin "1"
-		)
-		(pin "9"
-		)
-		(pin "10"
-		)
-		(pin "5"
-		)
-		(pin "7"
-		)
-		(instances
-			(project ""
-				(path "/7f2baae8-823e-4e28-b900-0a7e85154029"
-					(reference "T_GANFET")
-					(unit 1)
-				)
-			)
-		)
-	)
-	(symbol
 		(lib_id "Device:C")
 		(at 142.24 63.5 0)
@@
 	)
 	(symbol
+		(lib_id "EPC_FETs:EPC2066")
+		(at 54.61 115.57 270)
+		(mirror x)
+		(unit 1)
+		(exclude_from_sim no)
+		(in_bom yes)
+		(on_board yes)
+		(dnp no)
+		(property "Reference" "Q2"
+			(at 54.61 105.41 90)
+			(effects
+				(font
+					(size 1.27 1.27)
+				)
+			)
+		)
+		(property "Value" "EPC2066"
+			(at 54.61 107.95 90)
+			(effects
+				(font
+					(size 1.27 1.27)
+				)
+			)
+		)
+		(property "Footprint" "EPC_FETs:D0650"
+			(at 50.9524 109.6772 0)
+			(effects
+				(font
+					(size 1.27 1.27)
+				)
+				(hide yes)
+			)
+		)
+		(property "Datasheet" ""
+			(at 54.61 115.57 0)
+			(effects
+				(font
+					(size 1.27 1.27)
+				)
+				(hide yes)
+			)
+		)
+		(property "Description" "40V 1.1mE 90A"
+			(at 54.61 110.49 90)
+			(effects
+				(font
+					(size 1.27 1.27)
+				)
+			)
+		)
+		(pin "11"
+		)
+		(pin "1"
+		)
+		(pin "3"
+		)
+		(pin "23"
+		)
+		(pin "7"
+		)
+		(pin "24"
+		)
+		(pin "20"
+		)
+		(pin "4"
+		)
+		(pin "27"
+		)
+		(pin "19"
+		)
+		(pin "15"
+		)
+		(pin "28"
+		)
+		(pin "12"
+		)
+		(pin "16"
+		)
+		(pin "8"
+		)
+		(pin "10"
+		)
+		(pin "13"
+		)
+		(pin "14"
+		)
+		(pin "17"
+		)
+		(pin "18"
+		)
+		(pin "2"
+		)
+		(pin "21"
+		)
+		(pin "22"
+		)
+		(pin "25"
+		)
+		(pin "26"
+		)
+		(pin "29"
+		)
+		(pin "30"
+		)
+		(pin "5"
+		)
+		(pin "6"
+		)
+		(pin "9"
+		)
+		(instances
+			(project "GaN-LTC7891"
+				(path "/7f2baae8-823e-4e28-b900-0a7e85154029"
+					(reference "Q2")
+					(unit 1)
+				)
+			)
+		)
+	)
+	(symbol
 		(lib_id "Device:C")
 		(at 148.59 115.57 0)
@@
 					(unit 1)
 				)
-			)
-		)
-	)
-	(symbol
-		(lib_id "EPC_FETs:EPC2001C")
-		(at 54.61 115.57 270)
-		(mirror x)
-		(unit 1)
-		(exclude_from_sim no)
-		(in_bom yes)
-		(on_board yes)
-		(dnp no)
-		(property "Reference" "B_GANFET"
-			(at 50.546 106.68 90)
-			(effects
-				(font
-					(size 1.27 1.27)
-				)
-				(justify left)
-			)
-		)
-		(property "Value" "EPC2001C"
-			(at 50.292 111.506 90)
-			(effects
-				(font
-					(size 1.27 1.27)
-				)
-				(justify left)
-			)
-		)
-		(property "Footprint" "EPC_FETs:D0188"
-			(at 51.0032 109.22 0)
-			(effects
-				(font
-					(size 1.27 1.27)
-					(color 0 0 194 1)
-				)
-				(hide yes)
-			)
-		)
-		(property "Datasheet" ""
-			(at 54.61 115.57 0)
-			(effects
-				(font
-					(size 1.27 1.27)
-				)
-				(hide yes)
-			)
-		)
-		(property "Description" "100V 7mE 36A"
-			(at 48.768 109.474 90)
-			(effects
-				(font
-					(size 1.27 1.27)
-					(color 0 0 194 1)
-				)
-				(justify left)
-			)
-		)
-		(pin "6"
-		)
-		(pin "4"
-		)
-		(pin "2"
-		)
-		(pin "8"
-		)
-		(pin "3"
-		)
-		(pin "11"
-		)
-		(pin "1"
-		)
-		(pin "9"
-		)
-		(pin "10"
-		)
-		(pin "5"
-		)
-		(pin "7"
-		)
-		(instances
-			(project "GaN"
-				(path "/7f2baae8-823e-4e28-b900-0a7e85154029"
-					(reference "B_GANFET")
-					(unit 1)
-				)
