File: Si-LTC7800/Si-LTC7800.kicad_pcb (KiCad board)
At the start: 2 copper layers, 40 parts, among them Q1 BSC100N06LS3_G, Q2 BSC100N06LS3_G, U1 LTC7800HUDC_PBF

Commit message: connections and such
Parts:
- moved CSENSE 9.52 mm to (154.6, 138.3)
- moved CSENSE_EX1 6.38 mm to (154.6, 140.5)
- moved C5_EX1 5.68 mm to (127.3, 146.6), turned to 180 degrees
- moved R7 4.96 mm to (158.4, 143.7)
- moved R6 4.82 mm to (157.6, 141.8), turned to -45 degrees
- moved VSource_GND1 4.77 mm to (147.9, 152.8)
- moved R5 3.65 mm to (159.1, 143.7), turned to 90 degrees
- moved C5 3.39 mm to (127.3, 144.5), turned to 180 degrees
- moved C1_EX1 3.32 mm to (124.3, 132.9)
- moved C1 3.32 mm to (124.3, 134.9)
- moved C6_EX1 2.36 mm to (127.3, 141.5)
- moved C6 2.32 mm to (127.3, 139.5)
- moved R9 2.26 mm to (127.3, 143.0)
- moved COUT1 1.93 mm to (158.1, 129.5)
- moved RLOAD1 1.93 mm to (158.0, 131.7)
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- renumbered CSENSE1 to CSENSE
Routing:
- net /VFB: track 2.46 -> 30.4 mm, vias 1 -> 2
- net /Vout: track 26.0 -> 6.03 mm, vias 2 -> 1
- net /ITH: track 0.00 -> 11.3 mm, vias 0 -> 2
- net Net-(C5-Pad2): track 0.00 -> 3.70 mm
- net Net-(U1-TRACK/SS): track 8.68 -> 5.28 mm
- net /SENSE+: track 22.5 -> 24.7 mm
- net Net-(U1-FREQ): track 2.38 -> 1.25 mm
- net Net-(U1-PGOOD): track 3.69 -> 2.80 mm

Commit message: GaN PCB update
Parts:
- Q1, Q2: footprint XT60PW-M:BSC100N06LS3G -> Transistor_Power:BSC100N06LS3G
- U1: footprint Package_DFN_QFN:QFN50P400X300X80-21N -> Library:QFN50P400X300X80-21N
- moved VSource_GND1 4.77 mm to (148.0, 148.0)
- moved R2 4.00 mm to (122.6, 137.0)
- moved C1 2.96 mm to (121.4, 134.8)
- moved C1_EX1 2.96 mm to (121.4, 132.8)
- moved TP_VIN2 0.70 mm to (155.4, 154.0)
- renumbered CSENSE to CSENSE1
Routing:
- net /Vout: track 6.03 -> 37.2 mm, vias 1 -> 85
- net GND: track 0.00 -> 7.77 mm, vias 0 -> 77
- net /SENSE+: track 24.7 -> 19.4 mm
- net Net-(U1-FREQ): track 1.25 -> 5.42 mm
- net Net-(U1-TRACK/SS): track 5.28 -> 8.60 mm
- net /VIN: track 15.4 -> 15.9 mm
- added copper zone on B.Cu, net GND
- added copper zone on F.Cu, net GND
Other:
- board outline added: 54.8 x 47.8 mm
