File: Si-LTC7800-Alternate/Si-LTC7800-Alternate.kicad_pcb (KiCad board)
At the start: 2 copper layers, 54.8 x 47.8 mm, 40 parts, among them Q1 BSC100N06LS3_G, Q2 BSC100N06LS3_G, U1 LTC7800HUDC_PBF

Commit message: alternates
Parts:
- moved Q2 58.4 mm to (188.0, 119.6), turned to 90 degrees
- moved Q1 49.1 mm to (185.5, 127.2)
- moved TP_VIN1 15.4 mm to (137.5, 140.5)
- moved CinA1 7.25 mm to (131.8, 156.2)
- moved CinA1_EX1 7.25 mm to (127.8, 156.2)
- moved CinA2 7.25 mm to (129.8, 156.2)
- moved CinB1 7.25 mm to (133.8, 156.2)
- moved CinB1_EX1 7.25 mm to (125.8, 156.2)
- moved TP_VIN2 2.49 mm to (155.5, 151.5)
Routing:
- net /VIN: track 15.9 -> 105.4 mm
- net /BG: track 3.65 -> 88.2 mm, vias 0 -> 2
- net /SW: track 6.30 -> 58.2 mm
- net /TG: track 3.08 -> 55.0 mm, vias 0 -> 2
- net GND: vias 77 -> 69
Other:
- board size 54.8 x 47.8 mm -> 92.2 x 47.8 mm

Commit message: alternates good
Routing:
- net /BG: track 88.2 -> 89.1 mm
- net GND: vias 69 -> 99
